File: hardware/schem.sch (EAGLE design)
At the start: 18 parts, among them IC1 7805L, IC2 L298

Commit message: added current sensing
Connections:
- removed net N$1: IC2.SEN_A, IC2.SEN_B, R1.1
- net MOSI: now also IC2.SEN_A, IC2.SEN_B, R1.1
Other:
- moved on the sheet: R1
Changed lines of the file:
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@@
 <instance part="GND6" gate="1" x="182.88" y="10.16"/>
 <instance part="GND7" gate="1" x="127" y="-12.7"/>
-<instance part="R1" gate="G$1" x="170.18" y="12.7"/>
+<instance part="R1" gate="G$1" x="175.26" y="12.7"/>
 <instance part="DIODE1" gate="G$1" x="139.7" y="66.04" smashed="yes" rot="R90">
 <attribute name="NAME" x="139.2174" y="68.58" size="1.778" layer="95" rot="R90"/>
@@
 <pinref part="GND6" gate="1" pin="GND"/>
 <pinref part="R1" gate="G$1" pin="2"/>
-<wire x1="175.26" y1="12.7" x2="182.88" y2="12.7" width="0.1524" layer="91"/>
+<wire x1="180.34" y1="12.7" x2="182.88" y2="12.7" width="0.1524" layer="91"/>
 <junction x="182.88" y="12.7"/>
 </segment>
@@
 <label x="88.9" y="50.8" size="1.778" layer="95"/>
 </segment>
+<segment>
+<pinref part="IC2" gate="L298" pin="SEN_A"/>
+<pinref part="IC2" gate="L298" pin="SEN_B"/>
+<wire x1="162.56" y1="15.24" x2="162.56" y2="12.7" width="0.1524" layer="91"/>
+<wire x1="162.56" y1="12.7" x2="170.18" y2="12.7" width="0.1524" layer="91"/>
+<junction x="162.56" y="12.7"/>
+<pinref part="R1" gate="G$1" pin="1"/>
+<label x="165.1" y="12.7" size="1.778" layer="95"/>
+</segment>
 </net>
 <net name="MISO" class="0">
@@
 </segment>
 </net>
-<net name="N$1" class="0">
-<segment>
-<pinref part="IC2" gate="L298" pin="SEN_A"/>
-<pinref part="IC2" gate="L298" pin="SEN_B"/>
-<wire x1="162.56" y1="15.24" x2="162.56" y2="12.7" width="0.1524" layer="91"/>
-<wire x1="162.56" y1="12.7" x2="165.1" y2="12.7" width="0.1524" layer="91"/>
-<junction x="162.56" y="12.7"/>
-<pinref part="R1" gate="G$1" pin="1"/>
-</segment>
-</net>

Commit message: Changed Current Sense pin
Connections:
- net MOSI: now also IC2.INPUT2, IC2.INPUT3; no longer IC2.SEN_A, IC2.SEN_B, R1.1
- net SCK: now also IC2.SEN_A, IC2.SEN_B, R1.1; no longer IC2.INPUT2, IC2.INPUT3
Changed lines of the file:
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@@
 </segment>
 <segment>
-<pinref part="IC2" gate="L298" pin="SEN_A"/>
-<pinref part="IC2" gate="L298" pin="SEN_B"/>
-<wire x1="162.56" y1="15.24" x2="162.56" y2="12.7" width="0.1524" layer="91"/>
-<wire x1="162.56" y1="12.7" x2="170.18" y2="12.7" width="0.1524" layer="91"/>
-<junction x="162.56" y="12.7"/>
-<pinref part="R1" gate="G$1" pin="1"/>
-<label x="165.1" y="12.7" size="1.778" layer="95"/>
+<pinref part="IC2" gate="L298" pin="INPUT3"/>
+<pinref part="IC2" gate="L298" pin="INPUT2"/>
+<wire x1="132.08" y1="2.54" x2="132.08" y2="5.08" width="0.1524" layer="91"/>
+<wire x1="132.08" y1="5.08" x2="129.54" y2="5.08" width="0.1524" layer="91"/>
+<junction x="132.08" y="5.08"/>
+<label x="124.46" y="5.08" size="1.778" layer="95"/>
 </segment>
 </net>
@@
 </segment>
 <segment>
-<pinref part="IC2" gate="L298" pin="INPUT3"/>
-<pinref part="IC2" gate="L298" pin="INPUT2"/>
-<wire x1="132.08" y1="2.54" x2="132.08" y2="5.08" width="0.1524" layer="91"/>
-<wire x1="132.08" y1="5.08" x2="129.54" y2="5.08" width="0.1524" layer="91"/>
-<junction x="132.08" y="5.08"/>
-<label x="124.46" y="5.08" size="1.778" layer="95"/>
+<pinref part="IC2" gate="L298" pin="SEN_A"/>
+<pinref part="IC2" gate="L298" pin="SEN_B"/>
+<wire x1="162.56" y1="15.24" x2="162.56" y2="12.7" width="0.1524" layer="91"/>
+<wire x1="162.56" y1="12.7" x2="170.18" y2="12.7" width="0.1524" layer="91"/>
+<junction x="162.56" y="12.7"/>
+<pinref part="R1" gate="G$1" pin="1"/>
+<label x="165.1" y="12.7" size="1.778" layer="95"/>
 </segment>
 </net>

Commit message: Replaced diodes
Parts:
- DIODE1, DIODE2, DIODE3, DIODE4: value DIODE-ZENERPTH -> (none); device SparkFun-DiscreteSemi:DIODE-ZENERPTH -> diode:DIODE-DO41-7.6
Changed lines of the file:
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@@
 <part name="GND7" library="supply1" deviceset="GND" device=""/>
 <part name="R1" library="SparkFun-Passives" deviceset="RESISTOR" device="PTH-1/4W"/>
-<part name="DIODE1" library="SparkFun-DiscreteSemi" deviceset="DIODE-ZENER" device="PTH"/>
-<part name="DIODE2" library="SparkFun-DiscreteSemi" deviceset="DIODE-ZENER" device="PTH"/>
-<part name="DIODE3" library="SparkFun-DiscreteSemi" deviceset="DIODE-ZENER" device="PTH"/>
-<part name="DIODE4" library="SparkFun-DiscreteSemi" deviceset="DIODE-ZENER" device="PTH"/>
+<part name="DIODE1" library="diode" deviceset="DIODE-" device="DO41-7.6"/>
+<part name="DIODE2" library="diode" deviceset="DIODE-" device="DO41-7.6"/>
+<part name="DIODE3" library="diode" deviceset="DIODE-" device="DO41-7.6"/>
+<part name="DIODE4" library="diode" deviceset="DIODE-" device="DO41-7.6"/>
 <part name="P+8" library="supply1" deviceset="+12V" device=""/>
 <part name="GND8" library="supply1" deviceset="GND" device=""/>
